File: hdw/display_board/multidrop_display_board/Telemetry.sch (KiCad schematic (older format))
At the start: 0 parts

Commit message: more sch work
Parts:
- added C301, C302, C303: 0.1uF, Capacitors_SMD:C_0402, symbol Custom_Library:C_Custom
- added DOC301: 0x40, symbol Custom_Library:I2C_Address
- added DOC302: 0x18, symbol Custom_Library:I2C_Address
- added U301: INA219BxDCN, Package_TO_SOT_SMD:SOT-23-8, symbol Analog_ADC:INA219BxDCN
- added U302: MCP9804, Package_DFN_QFN:DFN-8-1EP_3x2mm_P0.5mm_EP1.3x1.5mm, symbol Sensor_Temperature:MCP9804_DFN
Connections:
- new net +3V3: C302.1, C303.1, U301.4 (VS), U302.8 (VDD)
- new net GND: C302.2, C303.2, U301.3 (GND), U301.7 (A0), U301.8 (A1), U302.4 (GND), U302.5 (A2), U302.6 (A1), U302.7 (A0), U302.9 (EP/GND)
- new net I2C_SCL: U301.5 (SCL), U302.2 (SCL)
- new net I2C_SDA: U301.6 (SDA), U302.1 (SDA)
- new net Telemetry_SNS+: C301.1, U301.1 (IN+)
- new net Telemetry_SNS-: C301.2, U301.2 (IN-)
- no-connect marks 0 -> 1
