File: hdw/display_board/multidrop_display_board/IO_Connectors.sch (KiCad schematic (older format))
At the start: 0 parts

Commit message: Added LED drivers, IO connectors to SCH
Parts:
- added C?: 10uF, Capacitors_SMD:C_0603, symbol Custom_Library:C_Custom
- added J?: Input Header, Pin_Headers:Pin_Header_Angled_2x16_Pitch2.54mm, symbol Connector_Generic:Conn_02x16_Odd_Even
- added J?: Output Socket, Socket_Strips:Socket_Strip_Angled_2x16_Pitch2.54mm, symbol Connector_Generic:Conn_02x16_Odd_Even
- added R?: 0.02, symbol Custom_Library:R_Custom
- added R? (x2): 10, Resistors_SMD:R_0402, symbol Custom_Library:R_Custom
Connections:
- new net +5V: C?.1, R?.1, R?.1
- new net +5VP: J?.10 (Pin_10), J?.10 (Pin_10), J?.2 (Pin_2), J?.2 (Pin_2), J?.4 (Pin_4), J?.4 (Pin_4), J?.6 (Pin_6), J?.6 (Pin_6), J?.8 (Pin_8), J?.8 (Pin_8), R?.1, R?.2
- new net EXT_RESET: J?.12 (Pin_12), J?.12 (Pin_12)
- new net GND: C?.2, J?.1 (Pin_1), J?.1 (Pin_1), J?.11 (Pin_11), J?.11 (Pin_11), J?.13 (Pin_13), J?.13 (Pin_13), J?.14 (Pin_14), J?.14 (Pin_14), J?.15 (Pin_15), J?.15 (Pin_15), J?.17 (Pin_17), J?.17 (Pin_17), J?.19 (Pin_19), J?.19 (Pin_19), J?.20 (Pin_20), J?.20 (Pin_20), J?.21 (Pin_21), J?.21 (Pin_21), J?.23 (Pin_23), J?.23 (Pin_23), J?.25 (Pin_25), J?.25 (Pin_25), J?.26 (Pin_26), J?.26 (Pin_26), J?.27 (Pin_27), J?.27 (Pin_27), J?.29 (Pin_29), J?.29 (Pin_29), J?.3 (Pin_3), J?.3 (Pin_3), J?.31 (Pin_31), J?.31 (Pin_31), J?.32 (Pin_32), J?.32 (Pin_32), J?.5 (Pin_5), J?.5 (Pin_5), J?.7 (Pin_7), J?.7 (Pin_7), J?.9 (Pin_9), J?.9 (Pin_9)
- new net RS485_CLK_SYNC+: J?.28 (Pin_28), J?.28 (Pin_28)
- new net RS485_CLK_SYNC-: J?.30 (Pin_30), J?.30 (Pin_30)
- new net RS485_RX+: J?.16 (Pin_16), J?.16 (Pin_16)
- new net RS485_RX-: J?.18 (Pin_18), J?.18 (Pin_18)
- new net RS485_TX+: J?.24 (Pin_24), J?.24 (Pin_24)
- new net RS485_TX-: J?.22 (Pin_22), J?.22 (Pin_22)
- new net Telemetry_SNS+: R?.2
- new net Telemetry_SNS-: R?.2
