File: hdw/display_board/multidrop_display_board/LED_Drivers.sch (KiCad schematic (older format))
At the start: 0 parts

Commit message: Added LED drivers, IO connectors to SCH
Parts:
- added Q? (x17): BSS214NW, Package_TO_SOT_SMD:SOT-323_SC-70, symbol Transistor_FET:BSS214NW
- added R? (x17): 10k, Resistors_SMD:R_0603, symbol Custom_Library:R_Custom
- added R? (x17): 120, symbol Custom_Library:R_Custom
- added R? (x17): 120, Resistors_SMD:R_0603, symbol Custom_Library:R_Custom
Connections:
- new net: Q?.1 (G), R?.1, R?.1 (x17)
- new net: Q?.3 (D), R?.2 (x17)
- new net GND: Q?.2 (S), Q?.2 (S), Q?.2 (S), Q?.2 (S), Q?.2 (S), Q?.2 (S), Q?.2 (S), Q?.2 (S), Q?.2 (S), Q?.2 (S), Q?.2 (S), Q?.2 (S), Q?.2 (S), Q?.2 (S), Q?.2 (S), Q?.2 (S), Q?.2 (S), R?.2, R?.2, R?.2, R?.2, R?.2, R?.2, R?.2, R?.2, R?.2, R?.2, R?.2, R?.2, R?.2, R?.2, R?.2, R?.2, R?.2
- new net SEGMENT_A: R?.1
- new net SEGMENT_A_DRIVE: R?.2
- new net SEGMENT_B: R?.1
- new net SEGMENT_B_DRIVE: R?.2
- new net SEGMENT_C: R?.1
- new net SEGMENT_C_DRIVE: R?.2
- new net SEGMENT_D: R?.1
- new net SEGMENT_DP: R?.1
- new net SEGMENT_DP_DRIVE: R?.2
- new net SEGMENT_D_DRIVE: R?.2
- new net SEGMENT_E: R?.1
- new net SEGMENT_E_DRIVE: R?.2
- new net SEGMENT_F: R?.1
- new net SEGMENT_F_DRIVE: R?.2
- new net SEGMENT_G: R?.1
- new net SEGMENT_G_DRIVE: R?.2
- new net SEGMENT_H: R?.1
- new net SEGMENT_H_DRIVE: R?.2
- new net SEGMENT_K: R?.1
- new net SEGMENT_K_DRIVE: R?.2
- new net SEGMENT_M: R?.1
- new net SEGMENT_M_DRIVE: R?.2
- new net SEGMENT_N: R?.1
- new net SEGMENT_N_DRIVE: R?.2
- new net SEGMENT_P: R?.1
- new net SEGMENT_P_DRIVE: R?.2
- new net SEGMENT_R: R?.1
- new net SEGMENT_R_DRIVE: R?.2
- new net SEGMENT_S: R?.1
- new net SEGMENT_S_DRIVE: R?.2
- new net SEGMENT_T: R?.1
- new net SEGMENT_T_DRIVE: R?.2
- new net SEGMENT_U: R?.1
- new net SEGMENT_U_DRIVE: R?.2
