File: hdw/display_board/multidrop_display_board/PIC18F.sch (KiCad schematic (older format))
At the start: 0 parts

Commit message: more sch work
Parts:
- added C?: 0.1uF, Capacitors_SMD:C_0603, symbol Custom_Library:C_Custom
- added C?: 10uF, Capacitors_SMD:C_0603, symbol Custom_Library:C_Custom
- added DOC501: Master, symbol Custom_Library:I2C_Address
- added R503, R504: 10k, Resistors_SMD:R_0603, symbol Custom_Library:R_Custom
- added U503: PIC18F27K40T-I_ML, Housings_DFN_QFN:QFN-28-1EP_6x6mm_Pitch0.65mm, symbol Custom_Library:PIC18(L)F27K40T-I_ML
Connections:
- new net +5V: C?.1, C?.1, R503.1, R504.1, U503.17 (VDD)
- new net GND: C?.2, C?.2, U503.16 (VSS), U503.29 (VSS), U503.5 (VSS)
- new net I2C_SCL: R503.2, U503.23 (RB5)
- new net I2C_SDA: R504.2, U503.22 (RB4)
- new net PIC18F_ICSPCLK: U503.24 (RB6/ICSPCLK)
- new net PIC18F_ICSPDAT: U503.25 (RB7/ICSPDAT)
- new net ~PIC18F_MCLR: U503.26 (RE3/~MCLR~/Vpp)
